File: full_board/red_line/red_line_v2/red_line_v2.kicad_pcb (KiCad board)
At the start: 2 copper layers, 171.8 x 202.3 mm, 122 parts, among them J2 Conn_01x15_Socket, J3 Conn_01x15_Socket, J4 USB_B_Micro, U1 MCP23S17T-E/SS, U2 MCP23S17T-E/SS, U3 MCP23S17T-E/SS

Commit message: add silkscreen, adjust layout
Parts:
- added G***: LOGO, demo.preety:sign, F.Cu at (156.2, 233.4)
- added G***: LOGO, demo.preety:mapagain, F.Cu at (198.4, 132.6)
- moved D23 69.8 mm to (271.0, 225.8), turned to -135 degrees
- moved D49 69.8 mm to (125.6, 40.6), turned to 45 degrees
- moved D15 67.0 mm to (235.2, 182.9), turned to -135 degrees
- moved D51 67.0 mm to (134.5, 40.8), turned to 45 degrees
- moved D50 66.5 mm to (125.8, 45.9), turned to 45 degrees
- moved D24 65.4 mm to (265.3, 225.9), turned to -135 degrees
- moved D52 64.2 mm to (134.4, 46.4), turned to 45 degrees
- moved D21 59.7 mm to (266.7, 204.8), turned to -135 degrees
- moved D11 59.5 mm to (214.6, 143.6), turned to -135 degrees
- moved D13 59.4 mm to (205.5, 160.1), turned to -135 degrees
- moved D17 59.4 mm to (249.1, 186.8), turned to -135 degrees
- moved D25 59.2 mm to (200.2, 172.5), turned to -135 degrees
- moved D19 59.2 mm to (257.9, 195.7), turned to -135 degrees
- moved R17 59.1 mm to (266.6, 140.7)
- moved R20 59.1 mm to (266.6, 151.6)
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Routing:
- net /LED29: track 88.3 -> 23.6 mm
- net Net-(D33-A): track 83.0 -> 20.7 mm
- net /LED31: track 74.4 -> 17.4 mm
- net Net-(D34-A): track 65.7 -> 13.3 mm
- net /LED32: track 72.4 -> 20.8 mm
- net /LED27: track 80.5 -> 31.8 mm
- net /LED33: track 59.5 -> 106.7 mm
- net /LED15: track 63.7 -> 109.8 mm
- net /LED37: track 50.5 -> 92.2 mm
- net Net-(D35-A): track 63.0 -> 21.4 mm
- net /LED25: track 88.4 -> 48.0 mm
- net /LED34: track 70.4 -> 109.8 mm
- net Net-(D29-A): track 126.9 -> 166.1 mm
- net /LED36: track 66.2 -> 104.3 mm
- net Net-(D27-A): track 111.7 -> 149.8 mm
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Other:
- board size 171.8 x 202.3 mm -> 178.7 x 219.7 mm
